Commit message: effort_joints

File: urdf/cart_assembly.urdf (robot description, URDF)
Before this commit: robot cart_assembly, 4 links, 3 joints
Joints:
- joint wheel_1_rot: type revolute -> continuous
- joint wheel_2_rot: type revolute -> continuous
- joint wheel_3_rot: type revolute -> continuous

Commit message: void

File: urdf/cart_assembly.urdf (robot description, URDF)
Before this commit: robot cart_assembly, 4 links, 3 joints
Links:
- link base_link: mass 11.6417381644856 -> 0.107381644856
