Commit message: update

File: urdf/main.xacro (robot description, xacro)
@@ -47,7 +47,7 @@
   <xacro:rim name="front" parent="base_link" xyz="0.095111 -0.054498 -0.093" rpy="-1.5708 0.70754 1.0472" GAZEBO_color = "Gazebo/Black"/>
  <!-- Laser -->
- <!-- <link name = "laser">
+ <link name = "laser">
     <visual>
-      <origin xyz="0 0 0.0" rpy="0 0 0" />
+      <origin xyz="0 0 0.1" rpy="0 0 0" />
       <geometry>
           <cylinder length="0.1" radius="0.01" />
@@ -61,5 +61,5 @@
     <parent link = "base_link"/>
     <child link = "laser"/>
-    <origin xyz="0 0 0.1" rpy="0 0 0"/>
-  </joint> -->
+    <origin xyz="0 0 0.5" rpy="0 0 0"/>
+  </joint>
 </robot>
